File: hardware/carSpd/carSpd.sch (EAGLE design)
At the start: 71 parts, among them IC1 DS3231/SO, IC2 CP2102, Q1 2n3904, U2 MP2307, U3 7805DT, U4 ATMEGA328P_TQFP, Y1 16MHZ, Y2 16mhz

Commit message: Replaced power regulator circuits
Parts:
- removed C20, C24, C25: 0.1uf, rcl:C-EUC0603K
- removed C22, C23: 18pf, rcl:C-EUC0603K
- removed DISPLAY: ERC1602-4SMD-LED, hybridair:ERC1602-4SMD-LED
- removed JP3: USBSMD, SparkFun-Connectors:USBSMD
- removed L2: 10uh, rcl:L-USL3225M
- removed R17: 47k, rcl:R-US_R0805
- removed R18: 2.7k, rcl:R-US_R0603
- removed U$2: DS1820, Ava:DS1820
- added C15: 0.1uf, rcl:C-EUC0603K
- added D7, D8: ZMM5V1, hybridair:ZMM5V1
- added IC3: DS3231/SO, adafruit:DS3231/SO
- added JP1: AVR_ICSP, SparkFun-Connectors:AVR_SPI_PRG_6TESTPOINTS
- added U1: ATMEGA328P_TQFP, SparkFun-DigitalIC:ATMEGA328P_TQFP
- C1: value 10uf -> 18pf
- C2: value 22uf -> 0.1uf
- C3: value 3.9nf -> 0.1uf
- C4: value 0.1uf -> 18pf
- C5: value 10nf -> 10uf; device rcl:C-EUC0805K -> rcl:C-EUC0603K
- C6: value 100uf -> 100nf; device ELL-i-Passives:CPOLD -> rcl:C-EUC0603K
- C7: value 10uf -> 22uf
- D4: value 5.1V -> DIODE-SCHOTTKY-BAT20J; device hybridair:ZMM5V1 -> SparkFun-DiscreteSemi:DIODE-SCHOTTKY-BAT20J
- D5: value 5.1V -> 1N4148; device hybridair:ZMM5V1 -> SparkFun-DiscreteSemi:DIODEBAS16
- D6: value 5.1V -> ZMM5V1
- IC1: value DS3231/SO -> MCP16301/H; device adafruit:DS3231/SO -> MCP16301:MCP16301/H
- JP2: value AVR_ICSP -> USBSMD; device SparkFun-Connectors:AVR_SPI_PRG_6TESTPOINTS -> SparkFun-Connectors:USBSMD
- L1: value CD54 -> 22uh; device inductor-sumida:CD54 -> rcl:L-USL3225M
- LED1: value (none) -> STATUS
- LED2: value (none) -> POWER
- LED5: value STATUS -> (none)
- LED6: value POWER -> (none)
- R12: value 4.7k -> 2.7k; device rcl:R-US_R0805 -> rcl:R-US_R0603
- R13: value 4.7k -> 10k; device rcl:R-US_R0805 -> rcl:R-US_R0603
- R14: value 270 -> 150
- R15, R16: value 47k -> 4.7k
- R2: value 100k -> 270; device rcl:R-US_R0805 -> rcl:R-US_R0603
- R3: value 6.8k -> 4.7k; device rcl:R-US_R0603 -> rcl:R-US_R0805
- R4: value 44.2k -> 4.7k; device rcl:R-US_R0603 -> rcl:R-US_R0805
- R5, R7: value 10k -> 47k; device rcl:R-US_R0603 -> rcl:R-US_R0805
- R6: value 4.7k -> 47k
- R8: value 150 -> 10k
- R9: value 4.7k -> 52.3k; device rcl:R-US_R0805 -> rcl:R-US_R0603
- S1: value SWITCH-MOMENTARY-2SMD-1101NE -> RESET
- S5: value RESET -> SWITCH-MOMENTARY-2SMD-1101NE
- SV1: device con-lsta:FE05W -> con-lsta:FE06W
- U2: value MP2307 -> (none); device hybridair:MP2307 -> SparkFun-IC-Power:V_REG_LM1117SOT223
- U3: value 7805DT -> ERC1602-4SMD-LED; device adafruit:7805DT -> hybridair:ERC1602-4SMD-LED
- U4: value ATMEGA328P_TQFP -> DS1820; device SparkFun-DigitalIC:ATMEGA328P_TQFP -> Ava:DS1820
- Y1: value 16MHZ -> 16mhz; device SparkFun-FreqCtrl:RESONATOR16MHZ -> SparkFun-FreqCtrl:CRYSTAL5X3
- Y2: value 16mhz -> 16MHZ; device SparkFun-FreqCtrl:CRYSTAL5X3 -> SparkFun-FreqCtrl:RESONATOR16MHZ
- renumbered C17 to C14, C18 to C13, C19 to C12
Connections:
- removed net N$1: C5.2, U2.BS
- removed net N$2: C5.1, L1.2, L2.2, U2.SW
- removed net N$3: R1.2, R4.2, U2.FB
- removed net N$5: C3.2, R3.2
- removed net N$6: C3.1, U2.COMP
- removed net N$7: C4.1, U2.SS
- removed net N$9: R2.1, U2.EN
- new net N$18: C6.1, D4.C, IC1.SW, L1.1
- new net N$19: C6.2, D5.C, IC1.BOOST
- new net N$25: C7.2, IC1.VFB, R8.1, R9.1
- net +12V: now also C5.1, IC1.EN, IC1.VIN, SV1.2; no longer C1.1, C6.+, R2.2, SV1.1, U3.VI
- net +5V: now also C15.1, C3.1, D5.A, IC3.VCC, JP1.2, JP2.VBUS, L1.2, R1.1, R12.2, R16.2, R3.1, R9.2, SV1.1, U1.AVCC, U1.VCC@4, U1.VCC@6, U2.OUT, U2.OUT@1, U3.PSB, U3.RS, U3.VDD, U3.XRESET, U4.VCC; no longer C20.1, C24.1, C25.1, DISPLAY.PSB, DISPLAY.RS, DISPLAY.VDD, DISPLAY.XRESET, IC1.VCC, JP2.2, JP3.VBUS, L1.1, L2.1, R11.1, R12.1, R13.1, R18.2, R6.2, U$2.VCC, U3.VO, U4.AVCC, U4.VCC@4, U4.VCC@6
- net D+: now also JP2.D+; no longer JP3.D+
- net D-: now also JP2.D-; no longer JP3.D-
- net GND: now also C15.2, C3.2, C4.1, C5.2, D7.A, D8.A, IC3.GND, IC3.NC, IC3.NC1, IC3.NC2, IC3.NC3, IC3.NC4, IC3.NC5, IC3.NC6, IC3.NC7, JP1.6, JP2.GND, LED5.C, R11.1, R2.2, R8.2, S1.1, S5.2, SV1.6, U1.AGND, U1.GND@3, U1.GND@5, U2.ADJ, U3.CSB, U3.LED-, U3.PSI2B, U3.VSS, U4.GND, Y2.2; no longer C20.2, C22.2, C23.1, C24.2, C25.2, C4.2, C6.-, C7.2, D5.A, DISPLAY.CSB, DISPLAY.LED-, DISPLAY.PSI2B, DISPLAY.VSS, IC1.NC, IC1.NC1, IC1.NC2, IC1.NC3, IC1.NC4, IC1.NC5, IC1.NC6, IC1.NC7, JP2.6, JP3.GND, LED1.C, R1.1, R14.2, R3.1, R7.1, S1.2, S5.1, SV1.5, U$2.GND, U2.GND, U3.GND, U4.AGND, U4.GND@3, U4.GND@5, Y1.2
- net INJ: now also R6.1, SV1.4; no longer R15.1, SV1.3
- net LED_PWM: now also JP1.4, R13.2, U1.PB3(MOSI/OC2); no longer JP2.4, R5.2, U4.PB3(MOSI/OC2)
- net LIGHTING: now also R7.1, SV1.5; no longer R17.1, SV1.4
- net N$11: now also R13.1; no longer R5.1
- net N$14: now also U3.VOUT; no longer DISPLAY.VOUT
- net N$15: now also R14.2, R15.2; no longer R8.2, R9.2
- net N$16: now also R14.1, U3.LED+; no longer DISPLAY.LED+, R8.1
- net N$20: now also U3.CAP1P; no longer DISPLAY.CAP1P
- net N$21: now also U3.CAP1N; no longer DISPLAY.CAP1N
- net N$22: now also JP1.1, U1.PB4(MISO); no longer JP2.1, U4.PB4(MISO)
- net N$23: now also LED5.A, LED6.A, R15.1; no longer LED1.A, LED2.A, R9.1
- net N$24: now also C1.1, U1.PB6(XTAL1/TOSC1), Y1.2, Y2.1; no longer C22.1, U4.PB6(XTAL1/TOSC1), Y1.1, Y2.2
- net N$26: now also JP1.3, LED1.A, U1.PB5(SCK); no longer JP2.3, LED5.A, U4.PB5(SCK)
- net N$27: now also IC3.VBAT; no longer IC1.VBAT
- net N$28: now also S2.1, U1.PD6(AIN0); no longer S1.1, U4.PD6(AIN0)
- net N$29: now also LED2.A, R12.1; no longer LED6.A, R18.1
- net N$30: now also D7.C, R6.2, U1.PD2(INT0), U1.PD3(INT1); no longer D5.C, R15.2, U4.PD2(INT0), U4.PD3(INT1)
- net N$31: now also D3.C, D8.C, R7.2, U1.PC0(ADC0); no longer D1.C, D4.C, R17.2, U4.PC0(ADC0)
- net N$32: now also LED1.C, R2.1; no longer LED5.C, R14.1
- net N$33: now also U1.PB0(ICP); no longer U4.PB0(ICP)
- net N$34: now also S4.1, U1.PD7(AIN1); no longer S2.1, U4.PD7(AIN1)
- net N$35: now also S5.1, U1.PB1(OC1A); no longer S4.1, U4.PB1(OC1A)
- net N$36: now also D1.C, R5.2, U1.PD5(T1); no longer D3.C, R16.2, U4.PD5(T1)
- net N$37: now also C4.2, U1.PB7(XTAL2/TOSC2), Y1.1, Y2.3; no longer C23.2, U4.PB7(XTAL2/TOSC2), Y1.3, Y2.1
- net N$4: now also R10.1; no longer R6.1
- net N$8: now also R11.2; no longer R7.2
- net RST: now also JP1.5, R1.2, S1.2, U1.PC6(/RESET); no longer JP2.5, R11.2, S5.2, U4.PC6(/RESET)
- net RX: now also U1.PD0(RXD); no longer U4.PD0(RXD)
- net SCL: now also IC3.SCL, R4.2, U1.PC5(ADC5/SCL), U3.SCL; no longer DISPLAY.SCL, IC1.SCL, R13.2, U4.PC5(ADC5/SCL)
- net SDA: now also IC3.SDA, R3.2, U1.PC4(ADC4/SDA), U3.SDA; no longer DISPLAY.SDA, IC1.SDA, R12.2, U4.PC4(ADC4/SDA)
- net TEMP: now also R16.1, U4.DQ; no longer R10.1, U$2.DQ
- net TX: now also U1.PD1(TXD); no longer U4.PD1(TXD)
- net VSS: now also R5.1, SV1.3; no longer R16.1, SV1.2
Other:
- note added: "Option 1 is a DC-DC buck regulator, and Option 2 is a linear regulator. Both are untested but should work. Option 1 is preferred due to its efficiency, but is more complex and untested, so it may not work in production. Option 2 is still untested, but it's simpler and should work if needed. Note: Option 2 uses C5 and C7 from Option 1."
- note removed: "12V comes from the car's accessory power rail, which is regulated down to 5V. The carSpd device itself shouldn't use more than 100ma."
- note removed: "ONLY USE ONE OPTION, DO NOT POPULATE BOTH AT ONCE"
- note removed: "Option 1 is an untested DC-DC buck regulator, and Option 2 is a tested, backup linear regulator circuit. Option 1 is preferred due to its efficiency, but is untested so it may not work in production. Option 2 is simpler, less efficient, but should work as expected."
- note removed: "Two inductor footprints are provided for part compatibility, use only one."
